File: esp32-wroom-sensor-board.kicad_pcb (KiCad board)
At the start: 2 copper layers, 99.6 x 99.3 mm, 57 parts, among them J3 USB_B_Micro, Q1 BSS138, Q2 BSS138, U3 TJA1051TK-3, U4 ESP32-WROOM-32, U5 CH340C

Commit message: minor fix
Parts:
- added R5: 10k, Resistor_SMD:R_0805_2012Metric_Pad1.20x1.40mm_HandSolder, F.Cu at (137.9, 84.6)
- moved C10 68.8 mm to (78.2, 49.8)
- moved C9 65.7 mm to (78.2, 52.3)
- moved C11 1.78 mm to (137.9, 79.5)
Routing:
- net +3.3V: track 252.5 -> 260.4 mm
- net /IO0: track 44.2 -> 51.9 mm
